Commit message: update 2/10

File: custom_arm.urdf (robot description, URDF)
Before this commit: robot test_arm, 4 links, 3 joints
Links:
- link elbow_link: geometry collision cylinder length=0.5 radius=0.075; visual cylinder length=0.5 radius=0.075
- link shoulder_link: geometry collision cylinder length=0.549 radius=0.075; visual cylinder length=0.549 radius=0.075
- link wrist_link: geometry collision cylinder length=0.125 radius=0.05; visual cylinder length=0.125 radius=0.05
Joints:
- joint armToEnd: origin xyz=0 0 0 rpy=0 0 0 -> xyz=0 0 2 rpy=0 0 0
- joint botToBase: origin xyz=0 0 0 rpy=0 0 0 -> xyz=0 0 0.2995 rpy=0 0 0
- joint topToBot: origin xyz=0 0 0 rpy=0 0 0 -> xyz=0 0 1 rpy=0 0 0
