Commit message: replacing old repo with working code

File: src/arm_description/urdf/custom_arm.urdf (robot description, URDF)
Before this commit: robot test_arm, 4 links, 3 joints
Links:
- added link base_endeffector, mass 0.032; collision box size=0.14 0.104 0.025; visual box size=0.14 0.104 0.025
- added link left_finger, mass 0.002; collision box size=0.03 0.1 0.05; visual box size=0.03 0.1 0.05
- added link little_link, mass 0.032; collision box size=0.05 0.05 0.05; visual box size=0.05 0.05 0.05
- added link right_finger, mass 0.032; collision box size=0.03 0.1 0.05; visual box size=0.03 0.1 0.05
- link base_link: mass 1 -> None
Joints:
- added joint endeffector: type continuous, parent wrist_link, child base_endeffector, origin xyz=0 0 0.125 rpy=0 0 0, axis 0 0 1
- added joint left_joint: type prismatic, parent base_endeffector, child left_finger, origin xyz=0.05 0 0.025 rpy=0 0 0, axis 1 0 0, limit lower=-0.035 upper=0.0 effort=100 velocity=5
- added joint right_joint: type prismatic, parent base_endeffector, child right_finger, origin xyz=-0.05 0 0.025 rpy=0 0 0, axis 1 0 0, limit lower=0.0 upper=0.035 effort=100 velocity=5
- added joint shoulderTolittle: type revolute, parent little_link, child shoulder_link, origin xyz=0 0 .05 rpy=0 0 0, axis 1 0 0, limit lower=0.0 upper=1.5707 effort=1000.0 velocity=0.5
- joint armToEnd: axis 0 0 1 -> 1 0 0; limit lower=0.0 upper=0.548 effort=1000.0 velocity=0.5 -> lower=0.0 upper=2.167 effort=1000.0 velocity=0.5
- joint botToBase: axis 1 0 0 -> 0 0 1; child shoulder_link -> little_link; limit lower=0.0 upper=0.548 effort=1000.0 velocity=0.5 -> (none); origin xyz=0 0 0.05 rpy=0 0 0 -> xyz=0 0 0.025 rpy=0 0 0; type revolute -> continuous
- joint topToBot: axis 0 0 1 -> 1 0 0; limit lower=0.0 upper=0.548 effort=1000.0 velocity=0.5 -> lower=0.0 upper=2.617 effort=1000.0 velocity=0.5; origin xyz=0 0 0.549 rpy=0 0 0 -> xyz=0 0 .549 rpy=0 0 0

Commit message: working arm

File: src/arm_description/urdf/custom_arm.urdf (robot description, URDF)
Before this commit: robot test_arm, 8 links, 7 joints
Links:
- added link world
Joints:
- added joint worldToBase: type fixed, parent world, child base_link, origin xyz=0 0 0.075 rpy=0 0 0, axis 0 0 1
- joint shoulderTolittle: origin xyz=0 0 .05 rpy=0 0 0 -> xyz=0 0 0.05 rpy=0 0 0

Commit message: can now launch rviz showing arm movement, gazebo launched without gui

File: src/arm_description/urdf/custom_arm.urdf (robot description, URDF)
Before this commit: robot test_arm, 9 links, 8 joints
Links:
- link base_endeffector: mass 0.032 -> 0.5
- link base_link: mass 1 -> 2
- link elbow_link: mass 0.3 -> 1
- link left_finger: mass 0.002 -> 0.5
- link little_link: mass 0.032 -> 5
- link right_finger: mass 0.032 -> 0.5
- link shoulder_link: mass 2.438816 -> 2.5
- link wrist_link: mass 0.032 -> 1
Joints:
- joint left_joint: limit lower=-0.035 upper=0.0 effort=100 velocity=5 -> lower=-0.035 upper=0.0 effort=100 velocity=${vel}
- joint right_joint: limit lower=0.0 upper=0.035 effort=100 velocity=5 -> lower=0.0 upper=0.035 effort=100 velocity=${vel}
